File: uCBoard/uCBoard.sch (EAGLE design)
At the start: 20 parts, among them X1 22-23-2041

Commit message: Committing gerber files
Parts:
- C1: device resistor:C-USC0805 -> rcl:C-USC1210
Changed lines of the file:
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@@
 <part name="R4" library="resistor" deviceset="R-US_" device="R0805" value="100k"/>
 <part name="R5" library="resistor" deviceset="R-US_" device="R0805" value="100k"/>
-<part name="C1" library="resistor" deviceset="C-US" device="C0805" value="220uF"/>
+<part name="C1" library="rcl" deviceset="C-US" device="C1210" value="220uF"/>
 <part name="L1" library="SparkFun-Passives" deviceset="INDUCTOR" device="0402" value="3.6nH"/>
 <part name="C2" library="resistor" deviceset="C-US" device="C0805" value="1pF"/>
